File: segundo_check/esquematico-check2/esquematico-check2.kicad_pcb (KiCad board)
At the start: 2 copper layers, 29 parts, among them J1 Conn_01x02, J2 Conn_01x02, Q1 BC547, Q2 BC547, Q3 BC547, Q4 BC557, Q5 BC557, Q6 MJE2955T, Q7 BC547, Q8 BC547, Q9 BC547, U1 TL431D

Commit message: Placa reglin terminada?
Parts:
- added R9: R, Resistor_THT:R_Axial_DIN0204_L3.6mm_D1.6mm_P5.08mm_Horizontal, F.Cu at (95.5, 75.5)
- C1: footprint Capacitor_THT:C_Rect_L9.0mm_W4.0mm_P7.50mm_MKT -> Capacitor_THT:C_Disc_D4.3mm_W1.9mm_P5.00mm
Connections:
- C1 pad 2: GND -> Net-(C1-Pad2)
Routing:
- net Net-(Q1-B): track 26.6 -> 33.3 mm
- net Net-(C1-Pad2): track 0.00 -> 3.83 mm
- net Net-(J1-Pin_2): track 85.5 -> 89.2 mm
- net Net-(JP2-B): track 24.3 -> 22.1 mm
- added copper zone on B.Cu, net GND
Other:
- board outline added: 100 x 50 mm

Commit message: Detalles previos a impresión de la placa
Parts:
- moved R4 10.1 mm to (112.0, 85.1), turned to 90 degrees
Routing:
- net Net-(Q7-B): track 25.1 -> 15.2 mm
- net Net-(J1-Pin_2): track 89.2 -> 86.3 mm
- net Net-(JP2-B): track 22.1 -> 20.3 mm
- net Net-(JP1-B): track 25.6 -> 26.2 mm
Other:
- board text added: "Martin Loñ Monti Del Rio"
Changed lines of the file:
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@@
 		(pad "1" thru_hole circle
 			(at 0 0)
-			(size 2 2)
+			(size 2.2 2.2)
 			(drill 1)
 			(layers "*.Cu" "*.Mask")
@@
 		(pad "1" thru_hole circle
 			(at 0 0)
-			(size 1.4 1.4)
+			(size 2 2)
 			(drill 0.8)
 			(layers "*.Cu" "*.Mask")
@@
 		(pad "2" thru_hole circle
 			(at 2.54 0)
-			(size 1.4 1.4)
+			(size 2 2)
 			(drill 0.8)
 			(layers "*.Cu" "*.Mask")
@@
 		(pad "1" thru_hole circle
 			(at 0 0)
-			(size 1.6 1.6)
+			(size 2 2)
 			(drill 0.8)
 			(layers "*.Cu" "*.Mask")
@@
 		(pad "2" thru_hole circle
 			(at 10.16 0)
-			(size 1.6 1.6)
+			(size 2 2)
 			(drill 0.8)
 			(layers "*.Cu" "*.Mask")
@@
 		(pad "1" thru_hole circle
 			(at 0 0)
-			(size 1.6 1.6)
+			(size 2 2)
 			(drill 0.8)
 			(layers "*.Cu" "*.Mask")
@@
 		(pad "2" thru_hole circle
 			(at 10.16 0)
-			(size 1.6 1.6)
+			(size 2 2)
 			(drill 0.8)
 			(layers "*.Cu" "*.Mask")
@@
 		(pad "1" thru_hole circle
 			(at 0 0 270)
-			(size 1.6 1.6)
+			(size 2 2)
 			(drill 0.8)
 			(layers "*.Cu" "*.Mask")
@@
 		(pad "2" thru_hole circle
 			(at 10.16 0 270)
-			(size 1.6 1.6)
+			(size 2 2)
 			(drill 0.8)
 			(layers "*.Cu" "*.Mask")
@@
 		(pad "1" thru_hole circle
 			(at 0 0 270)
-			(size 1.6 1.6)
+			(size 2 2)
 			(drill 0.8)
 			(layers "*.Cu" "*.Mask")
@@
 		(pad "2" thru_hole circle
 			(at 5 0 270)
-			(size 1.6 1.6)
+			(size 2 2)
 			(drill 0.8)
 			(layers "*.Cu" "*.Mask")
@@
 		(pad "1" thru_hole circle
 			(at 0 0)
-			(size 1.6 1.6)
+			(size 2 2)
 			(drill 0.8)
 			(layers "*.Cu" "*.Mask")
@@
 		(pad "2" thru_hole circle
 			(at 10.16 0)
-			(size 1.6 1.6)
+			(size 2 2)
 			(drill 0.8)
 			(layers "*.Cu" "*.Mask")
@@
 		(pad "1" thru_hole circle
 			(at 0 0)
-			(size 2 2)
+			(size 2.2 2.2)
 			(drill 1)
 			(layers "*.Cu" "*.Mask")
@@
 		(pad "1" thru_hole circle
 			(at 0 0)
-			(size 1.4 1.4)
+			(size 2 2)
 			(drill 0.8)
 			(layers "*.Cu" "*.Mask")
@@
 		(pad "2" thru_hole circle
 			(at 2.54 0)
-			(size 1.4 1.4)
+			(size 2 2)
 			(drill 0.8)
 			(layers "*.Cu" "*.Mask")
@@
 	(footprint "Resistor_THT:R_Axial_DIN0207_L6.3mm_D2.5mm_P10.16mm_Horizontal"
 		(layer "F.Cu")
-		(at 112 75 -90)
+		(at 112 85.08 90)
 		(descr "Resistor, Axial_DIN0207 series, Axial, Horizontal, pin pitch=10.16mm, 0.25W = 1/4W, length*diameter=6.3*2.5mm^2, http://cdn-reichelt.de/documents/datenblatt/B400/1_4W%23YAG.pdf")
 		(tags "Resistor Axial_DIN0207 series Axial Horizontal pin pitch 10.16mm 0.25W = 1/4W length 6.3mm diameter 2.5mm")
@@
 		(attr through_hole)
 		(fp_line
-			(start 1.04 0)
-			(end 1.81 0)
+			(start 9.12 0)
+			(end 8.35 0)
 			(stroke
 				(width 0.12)
@@
 		)
 		(fp_line
-			(start 9.12 0)
-			(end 8.35 0)
+			(start 1.04 0)
+			(end 1.81 0)
 			(stroke
 				(width 0.12)
@@
 		)
 		(fp_line
-			(start 0 0)
-			(end 1.93 0)
+			(start 10.16 0)
+			(end 8.23 0)
 			(stroke
 				(width 0.1)
@@
 		)
 		(fp_line
-			(start 10.16 0)
-			(end 8.23 0)
+			(start 0 0)
+			(end 1.93 0)
 			(stroke
 				(width 0.1)
@@
 		)
 		(pad "1" thru_hole circle
-			(at 0 0 270)
-			(size 1.6 1.6)
+			(at 0 0 90)
+			(size 2 2)
 			(drill 0.8)
 			(layers "*.Cu" "*.Mask")
@@
 		)
 		(pad "2" thru_hole circle
-			(at 10.16 0 270)
-			(size 1.6 1.6)
+			(at 10.16 0 90)
+			(size 2 2)
 			(drill 0.8)
 			(layers "*.Cu" "*.Mask")
@@
 		(pad "1" thru_hole circle
 			(at 0 0 270)
-			(size 1.6 1.6)
+			(size 2 2)
 			(drill 0.8)
 			(layers "*.Cu" "*.Mask")
@@
 		(pad "2" thru_hole circle
 			(at 10.16 0 270)
-			(size 1.6 1.6)
+			(size 2 2)
 			(drill 0.8)
 			(layers "*.Cu" "*.Mask")
@@
 		(pad "1" thru_hole circle
 			(at 0 0 270)
-			(size 1.4 1.4)
+			(size 2 2)
 			(drill 0.8)
 			(layers "*.Cu" "*.Mask")
@@
 		(pad "2" thru_hole circle
 			(at 2.54 0 270)
-			(size 1.4 1.4)
+			(size 2 2)
 			(drill 0.8)
 			(layers "*.Cu" "*.Mask")
@@
 		(pad "2" thru_hole circle
 			(at 0 5.08 180)
-			(size 2.8 2.8)
+			(size 3 3)
 			(drill 1.75)
 			(layers "*.Cu" "*.Mask")
@@
 		(pad "1" thru_hole rect
 			(at 0 0 270)
-			(size 1.5 1.5)
+			(size 1.7 1.7)
 			(drill 0.8)
 			(layers "*.Cu" "*.Mask")
@@
 		(pad "2" thru_hole circle
 			(at 2.54 0 270)
-			(size 1.5 1.5)
+			(size 2 2)
 			(drill 0.8)
 			(layers "*.Cu" "*.Mask")
@@
 		(pad "3" thru_hole circle
 			(at 5.08 0 270)
-			(size 1.5 1.5)
+			(size 2 2)
 			(drill 0.8)
 			(layers "*.Cu" "*.Mask")
@@
 		(pad "1" thru_hole circle
 			(at 0 0 270)
-			(size 1.4 1.4)
+			(size 2 2)
 			(drill 0.8)
 			(layers "*.Cu" "*.Mask")
@@
 		(pad "2" thru_hole circle
 			(at 2.54 0 270)
-			(size 1.4 1.4)
+			(size 2 2)
 			(drill 0.8)
 			(layers "*.Cu" "*.Mask")
@@
 		(pad "1" thru_hole circle
 			(at 0 0 90)
-			(size 1.4 1.4)
+			(size 2 2)
 			(drill 0.7)
 			(layers "*.Cu" "*.Mask")
@@
 		(pad "2" thru_hole circle
 			(at 5.08 0 90)
-			(size 1.4 1.4)
+			(size 2 2)
 			(drill 0.7)
 			(layers "*.Cu" "*.Mask")
@@
 		(pad "1" thru_hole circle
 			(at 0 0 270)
-			(size 1.6 1.6)
+			(size 2 2)
 			(drill 0.8)
 			(layers "*.Cu" "*.Mask")
@@
 		(pad "2" thru_hole circle
 			(at 10.16 0 270)
-			(size 1.6 1.6)
+			(size 2 2)
 			(drill 0.8)
 			(layers "*.Cu" "*.Mask")
@@
 		(pad "1" thru_hole circle
 			(at 0 0 270)
-			(size 1.6 1.6)
+			(size 2 2)
 			(drill 0.8)
 			(layers "*.Cu" "*.Mask")
@@
 		(pad "2" thru_hole circle
 			(at 10.16 0 270)
-			(size 1.6 1.6)
+			(size 2 2)
 			(drill 0.8)
 			(layers "*.Cu" "*.Mask")
@@
 		(pad "1" thru_hole rect
 			(at 0 0)
-			(size 1.5 1.5)
+			(size 1.7 1.7)
 			(drill 0.8)
 			(layers "*.Cu" "*.Mask")
@@
 		(pad "2" thru_hole circle
 			(at 2.54 0)
-			(size 1.5 1.5)
+			(size 2 2)
 			(drill 0.8)
 			(layers "*.Cu" "*.Mask")
@@
 		(pad "3" thru_hole circle
 			(at 5.08 0)
-			(size 1.5 1.5)
+			(size 2 2)
 			(drill 0.8)
 			(layers "*.Cu" "*.Mask")
@@
 		(pad "2" thru_hole circle
 			(at 0 5.08 180)
-			(size 2.8 2.8)
+			(size 3 3)
 			(drill 1.75)
 			(layers "*.Cu" "*.Mask")
@@
 		(layer "Edge.Cuts")
 	)
+	(gr_text "Martin\nLoñ\nMonti\nDel Rio"
+		(at 134 73 0)
+		(layer "B.Cu")
+		(effects
+			(font
+				(size 1.5 1.5)
+				(thickness 0.3)
+				(bold yes)
+			)
+			(justify left bottom mirror)
+		)
+	)
 	(segment
 		(start 130 91.5)
@@
 	)
 	(segment
-		(start 112 75)
-		(end 112 76.5)
-		(width 0.5)
-		(layer "B.Cu")
-		(net 5)
-	)
-	(segment
-		(start 108 84.5)
-		(end 111.5 88)
-		(width 0.5)
-		(layer "B.Cu")
-		(net 5)
-	)
-	(segment
-		(start 112 76.5)
-		(end 110 78.5)
+		(start 113.5 85.08)
+		(end 112 85.08)
 		(width 0.5)
 		(layer "B.Cu")
@@
 	)
 	(segment
-		(start 108 78.5)
-		(end 108 84.5)
-		(width 0.5)
-		(layer "B.Cu")
-		(net 5)
-	)
-	(segment
-		(start 110 78.5)
-		(end 108 78.5)
+		(start 105.42 78.5)
+		(end 105.14 78.5)
 		(width 0.5)
 		(layer "B.Cu")
@@
 	)
 	(segment
-		(start 111.5 88)
-		(end 116.42 88)
+		(start 112 85.08)
+		(end 105.42 78.5)
 		(width 0.5)
 		(layer "B.Cu")
@@
 	)
 	(segment
-		(start 108 78.5)
-		(end 105.14 78.5)
+		(start 116.42 88)
+		(end 113.5 85.08)
 		(width 0.5)
 		(layer "B.Cu")
@@
 	)
 	(segment
-		(start 55.5 61)
-		(end 64.08 52.42)
-		(width 1.5)
-		(layer "B.Cu")
-		(net 6)
-	)
-	(segment
-		(start 64.08 52.42)
-		(end 75 52.42)
+		(start 75 52.42)
+		(end 69.08 52.42)
 		(width 1.5)
 		(layer "B.Cu")
@@
 	)
 	(segment
-		(start 55.5 71.465)
-		(end 55.5 61)
+		(start 69.08 52.42)
+		(end 55.5 66)
+		(width 1.5)
+		(layer "B.Cu")
+		(net 6)
+	)
+	(segment
+		(start 55.5 66)
+		(end 55.5 71.465)
 		(width 1.5)
 		(layer "B.Cu")
@@
 	)
 	(segment
+		(start 98.79 66)
+		(end 110.02066 66)
+		(width 0.5)
+		(layer "B.Cu")
+		(net 12)
+	)
+	(segment
 		(start 99 66.21)
 		(end 98.79 66)
@@
 	)
 	(segment
-		(start 108.96 66)
-		(end 110.96 64)
+		(start 110.02066 66)
+		(end 110.96 65.06066)
 		(width 0.5)
 		(layer "B.Cu")
@@
 	)
 	(segment
-		(start 99 69.75)
-		(end 99 66.21)
+		(start 110.96 65.06066)
+		(end 110.96 64)
 		(width 0.5)
 		(layer "B.Cu")
@@
 	)
 	(segment
-		(start 98.79 66)
-		(end 108.96 66)
+		(start 99 69.75)
+		(end 99 66.21)
 		(width 0.5)
 		(layer "B.Cu")
@@
 	)
 	(segment
-		(start 116.5 80.66)
-		(end 112 85.16)
-		(width 1.5)
+		(start 112 74.92)
+		(end 116.37 74.92)
+		(width 0.5)
+		(layer "B.Cu")
+		(net 13)
+	)
+	(segment
+		(start 116.37 74.92)
+		(end 116.5 74.79)
+		(width 0.5)
 		(layer "B.Cu")
 		(net 13)
