File: cuarto_check/cuarto_check_oscilador/cuarto_check_oscilador.kicad_sch (KiCad schematic)
At the start: 19 parts, among them J1 Screw_Terminal_01x02, J2 Screw_Terminal_01x02, J3 Screw_Terminal_01x02, U1 LM393, U2 TL072

Commit message: Fin? diseño placa oscilador
Parts:
- removed C3: 100n, Capacitor_THT:C_Disc_D4.3mm_W1.9mm_P5.00mm, symbol Device:C
Changed lines of the file:
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@@
-	)
-	(junction
-		(at 129.54 20.32)
-		(diameter 0)
-		(color 0 0 0 0)
 	)
 	(junction
@@
 		(color 0 0 0 0)
 	)
-	(junction
-		(at 129.54 35.56)
-		(diameter 0)
-		(color 0 0 0 0)
-	)
 	(wire
 		(pts
@@
 	(wire
 		(pts
-			(xy 121.92 35.56) (xy 129.54 35.56)
-		)
-		(stroke
-			(width 0)
-			(type default)
-		)
-	)
-	(wire
-		(pts
 			(xy 85.09 76.2) (xy 88.9 76.2)
 		)
@@
 	(wire
 		(pts
-			(xy 121.92 24.13) (xy 121.92 20.32)
-		)
-		(stroke
-			(width 0)
-			(type default)
-		)
-	)
-	(wire
-		(pts
 			(xy 238.76 115.57) (xy 236.22 115.57)
 		)
@@
 	(wire
 		(pts
-			(xy 121.92 20.32) (xy 129.54 20.32)
-		)
-		(stroke
-			(width 0)
-			(type default)
-		)
-	)
-	(wire
-		(pts
 			(xy 109.22 50.8) (xy 109.22 60.96)
 		)
@@
 		(pts
 			(xy 167.64 76.2) (xy 172.72 76.2)
-		)
-		(stroke
-			(width 0)
-			(type default)
-		)
-	)
-	(wire
-		(pts
-			(xy 121.92 31.75) (xy 121.92 35.56)
 		)
 		(stroke
@@
 					(unit 1)
 				)
-			)
-		)
-	)
-	(symbol
-		(lib_id "Device:C")
-		(at 121.92 27.94 180)
-		(unit 1)
-		(exclude_from_sim no)
-		(in_bom yes)
-		(on_board yes)
-		(dnp no)
-		(fields_autoplaced yes)
-		(property "Reference" "C3"
-			(at 125.73 26.6699 0)
-			(effects
-				(font
-					(size 1.27 1.27)
-				)
-				(justify right)
-			)
-		)
-		(property "Value" "100n"
-			(at 125.73 29.2099 0)
-			(effects
-				(font
-					(size 1.27 1.27)
-				)
-				(justify right)
-			)
-		)
-		(property "Footprint" "Capacitor_THT:C_Disc_D4.3mm_W1.9mm_P5.00mm"
-			(at 120.9548 24.13 0)
-			(effects
-				(font
-					(size 1.27 1.27)
-				)
-				(hide yes)
-			)
-		)
-		(property "Datasheet" "~"
-			(at 121.92 27.94 0)
-			(effects
-				(font
-					(size 1.27 1.27)
-				)
-				(hide yes)
-			)
-		)
-		(property "Description" "Unpolarized capacitor"
-			(at 121.92 27.94 0)
-			(effects
-				(font
-					(size 1.27 1.27)
-				)
-				(hide yes)
-			)
-		)
-		(pin "1"
-		)
-		(pin "2"
-		)
-		(instances
-			(project "cuarto_check_oscilador"
-				(path "/f1d7cffb-e76c-49bb-8693-53407790405e"
-					(reference "C3")
-					(unit 1)
-				)

Commit message: matenme porfa
Parts:
- added C3: 100n, Capacitor_THT:C_Disc_D4.3mm_W1.9mm_P5.00mm, symbol Device:C
Connections:
- net GND: now also U1.4 (V-), U2.4 (V-), C3.1; no longer U1.8 (V+), U2.8 (V+)
- net Vin: now also U1.8 (V+), U2.8 (V+), C3.2; no longer U1.4 (V-), U2.4 (V-)
Other:
- moved on the sheet: C2
Changed lines of the file:
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@@
+	)
+	(junction
+		(at 129.54 35.56)
+		(diameter 0)
+		(color 0 0 0 0)
+	)
+	(junction
+		(at 143.51 35.56)
+		(diameter 0)
+		(color 0 0 0 0)
 	)
 	(junction
@@
 	)
 	(junction
-		(at 143.51 20.32)
-		(diameter 0)
-		(color 0 0 0 0)
-	)
-	(junction
 		(at 105.41 73.66)
 		(diameter 0)
@@
 	)
 	(junction
+		(at 143.51 20.32)
+		(diameter 0)
+		(color 0 0 0 0)
+	)
+	(junction
 		(at 109.22 73.66)
 		(diameter 0)
@@
 	)
 	(junction
-		(at 143.51 35.56)
+		(at 129.54 20.32)
 		(diameter 0)
 		(color 0 0 0 0)
@@
 	(wire
 		(pts
+			(xy 121.92 35.56) (xy 129.54 35.56)
+		)
+		(stroke
+			(width 0)
+			(type default)
+		)
+	)
+	(wire
+		(pts
 			(xy 167.64 76.2) (xy 162.56 76.2)
 		)
@@
 	(wire
 		(pts
-			(xy 153.67 31.75) (xy 153.67 35.56)
+			(xy 151.13 31.75) (xy 151.13 35.56)
 		)
 		(stroke
@@
 	(wire
 		(pts
+			(xy 121.92 31.75) (xy 121.92 35.56)
+		)
+		(stroke
+			(width 0)
+			(type default)
+		)
+	)
+	(wire
+		(pts
+			(xy 121.92 24.13) (xy 121.92 20.32)
+		)
+		(stroke
+			(width 0)
+			(type default)
+		)
+	)
+	(wire
+		(pts
 			(xy 57.15 74.93) (xy 57.15 83.82)
 		)
@@
 	(wire
 		(pts
-			(xy 129.54 39.37) (xy 129.54 35.56)
-		)
-		(stroke
-			(width 0)
-			(type default)
-		)
-	)
-	(wire
-		(pts
 			(xy 85.09 86.36) (xy 85.09 88.9)
 		)
@@
 	(wire
 		(pts
+			(xy 121.92 20.32) (xy 129.54 20.32)
+		)
+		(stroke
+			(width 0)
+			(type default)
+		)
+	)
+	(wire
+		(pts
 			(xy 256.54 110.49) (xy 256.54 118.11)
 		)
@@
 	(wire
 		(pts
+			(xy 129.54 35.56) (xy 129.54 39.37)
+		)
+		(stroke
+			(width 0)
+			(type default)
+		)
+	)
+	(wire
+		(pts
 			(xy 173.99 81.28) (xy 173.99 106.68)
 		)
@@
 	(wire
 		(pts
-			(xy 153.67 24.13) (xy 153.67 20.32)
+			(xy 151.13 24.13) (xy 151.13 20.32)
 		)
 		(stroke
@@
 	(wire
 		(pts
-			(xy 143.51 35.56) (xy 153.67 35.56)
+			(xy 143.51 35.56) (xy 151.13 35.56)
 		)
 		(stroke
@@
 	(wire
 		(pts
-			(xy 143.51 20.32) (xy 153.67 20.32)
+			(xy 143.51 20.32) (xy 151.13 20.32)
 		)
 		(stroke
@@
 	(symbol
 		(lib_id "Comparator:LM393")
-		(at 146.05 27.94 0)
-		(mirror x)
+		(at 140.97 27.94 0)
+		(mirror y)
 		(unit 3)
 		(exclude_from_sim no)
@@
 		(dnp no)
 		(property "Reference" "U1"
-			(at 146.05 38.1 0)
+			(at 140.97 17.78 0)
 			(effects
 				(font
@@
 		)
 		(property "Value" "LM393"
-			(at 146.05 35.56 0)
+			(at 140.97 20.32 0)
 			(effects
 				(font
@@
 		)
 		(property "Footprint" "Package_DIP:DIP-8_W7.62mm_LongPads"
-			(at 146.05 27.94 0)
+			(at 140.97 27.94 0)
 			(effects
 				(font
@@
 		)
 		(property "Datasheet" "http://www.ti.com/lit/ds/symlink/lm393.pdf"
-			(at 146.05 27.94 0)
+			(at 140.97 27.94 0)
 			(effects
 				(font
@@
 		)
 		(property "Description" "Low-Power, Low-Offset Voltage, Dual Comparators, DIP-8/SOIC-8/TO-99-8"
-			(at 146.05 27.94 0)
+			(at 140.97 27.94 0)
 			(effects
 				(font
@@
 	(symbol
 		(lib_id "Amplifier_Operational:TL072")
-		(at 132.08 27.94 0)
-		(mirror x)
+		(at 127 27.94 0)
+		(mirror y)
 		(unit 3)
 		(exclude_from_sim no)
@@
 		(dnp no)
 		(property "Reference" "U2"
-			(at 132.08 38.1 0)
+			(at 127 17.78 0)
 			(effects
 				(font
@@
 		)
 		(property "Value" "TL072"
-			(at 132.08 35.56 0)
+			(at 127 20.32 0)
 			(effects
 				(font
@@
 		)
 		(property "Footprint" "Package_DIP:DIP-8_W7.62mm_LongPads"
-			(at 132.08 27.94 0)
+			(at 127 27.94 0)
 			(effects
 				(font
@@
 		)
 		(property "Datasheet" "http://www.ti.com/lit/ds/symlink/tl071.pdf"
-			(at 132.08 27.94 0)
+			(at 127 27.94 0)
 			(effects
 				(font
@@
 		)
 		(property "Description" "Dual Low-Noise JFET-Input Operational Amplifiers, DIP-8/SOIC-8"
-			(at 132.08 27.94 0)
+			(at 127 27.94 0)
 			(effects
 				(font
@@
 	)
 	(symbol
+		(lib_id "Device:C")
+		(at 121.92 27.94 180)
+		(unit 1)
+		(exclude_from_sim no)
+		(in_bom yes)
+		(on_board yes)
+		(dnp no)
+		(fields_autoplaced yes)
+		(property "Reference" "C3"
+			(at 125.73 26.6699 0)
+			(effects
+				(font
+					(size 1.27 1.27)
+				)
+				(justify right)
+			)
+		)
+		(property "Value" "100n"
+			(at 125.73 29.2099 0)
+			(effects
+				(font
+					(size 1.27 1.27)
+				)
+				(justify right)
+			)
+		)
+		(property "Footprint" "Capacitor_THT:C_Disc_D4.3mm_W1.9mm_P5.00mm"
+			(at 120.9548 24.13 0)
+			(effects
+				(font
+					(size 1.27 1.27)
+				)
+				(hide yes)
+			)
+		)
+		(property "Datasheet" "~"
+			(at 121.92 27.94 0)
+			(effects
+				(font
+					(size 1.27 1.27)
+				)
+				(hide yes)
+			)
+		)
+		(property "Description" "Unpolarized capacitor"
+			(at 121.92 27.94 0)
+			(effects
+				(font
+					(size 1.27 1.27)
+				)
+				(hide yes)
+			)
+		)
+		(pin "1"
+		)
+		(pin "2"
+		)
+		(instances
+			(project "cuarto_check_oscilador"
+				(path "/f1d7cffb-e76c-49bb-8693-53407790405e"
+					(reference "C3")
+					(unit 1)
+				)
+			)
+		)
+	)
+	(symbol
 		(lib_id "Connector:Screw_Terminal_01x02")
 		(at 255.27 72.39 0)
@@
 	(symbol
 		(lib_id "Device:C")
-		(at 153.67 27.94 180)
+		(at 151.13 27.94 180)
 		(unit 1)
 		(exclude_from_sim no)
@@
 		(fields_autoplaced yes)
 		(property "Reference" "C2"
-			(at 157.48 26.6699 0)
+			(at 154.94 26.6699 0)
 			(effects
 				(font
@@
 		)
 		(property "Value" "100n"
-			(at 157.48 29.2099 0)
+			(at 154.94 29.2099 0)
 			(effects
 				(font
@@
 		)
 		(property "Footprint" "Capacitor_THT:C_Disc_D4.3mm_W1.9mm_P5.00mm"
-			(at 152.7048 24.13 0)
+			(at 150.1648 24.13 0)
 			(effects
 				(font
@@
 		)
 		(property "Datasheet" "~"
-			(at 153.67 27.94 0)
+			(at 151.13 27.94 0)
 			(effects
 				(font
@@
 		)
 		(property "Description" "Unpolarized capacitor"
-			(at 153.67 27.94 0)
-			(effects
-				(font
+			(at 151.13 27.94 0)
+			(effects
+				(font
