File: cuarto_check/cuarto_check_oscilador/cuarto_check_oscilador.kicad_pcb (KiCad board)
At the start: 2 copper layers, 60 x 60 mm, 19 parts, among them J1 Screw_Terminal_01x02, J2 Screw_Terminal_01x02, J3 Screw_Terminal_01x02, U1 LM393, U2 TL072

Commit message: Fin? diseño placa oscilador
Parts:
- removed C3: 100n, Capacitor_THT:C_Disc_D4.3mm_W1.9mm_P5.00mm
- moved TP3 72.0 mm to (83.6, 69.9)
- moved R2 66.9 mm to (54.0, 57.9), turned to 0 degrees
- moved J2 61.6 mm to (93.6, 70.4), turned to 0 degrees
- moved R5 61.3 mm to (88.1, 56.8), turned to -90 degrees
- moved C2 44.7 mm to (66.5, 80.0), turned to 90 degrees
- moved TP1 41.9 mm to (59.6, 61.4)
- moved JP1 39.6 mm to (86.1, 77.9)
- moved R4 36.8 mm to (64.1, 60.8)
- moved RV2 33.1 mm to (95.6, 88.0), turned to -90 degrees
- moved TP2 27.5 mm to (62.5, 85.5)
- moved J1 26.2 mm to (55.6, 75.4)
- moved J3 18.1 mm to (87.1, 88.9)
- moved R3 16.1 mm to (69.5, 76.9), turned to 0 degrees
- moved U2 5.98 mm to (76.4, 82.6)
- moved C1 5.02 mm to (81.6, 80.4)
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Routing:
- net Vin: track 0.54 -> 125.8 mm
- net Offset: track 12.8 -> 31.4 mm
- net Net-(U1A-+): track 0.00 -> 18.4 mm
- net Vout: track 0.00 -> 16.8 mm
- net DCycle: track 0.00 -> 12.6 mm
- net Net-(JP1-C): track 0.00 -> 11.7 mm
- net Net-(R1-Pad2): track 7.93 -> 19.0 mm
- net Net-(U1B--): track 15.8 -> 25.4 mm
- net ExtDCycle: track 0.00 -> 6.37 mm
- net Net-(U2B--): track 0.00 -> 2.54 mm
- net Net-(U2A--): track 33.1 -> 35.4 mm
- added copper zone on B.Cu, net GND
Other:
- board size 60 x 60 mm -> 50 x 50 mm
- board text added: "Martín Loñ Monti Del Rio"

Commit message: matenme porfa
Parts:
- added C3: 100n, Capacitor_THT:C_Disc_D4.3mm_W1.9mm_P5.00mm, F.Cu at (83.5, 70.5)
- moved C2 15.7 mm to (80.0, 88.0), turned to -90 degrees
- moved J1 7.32 mm to (53.9, 82.5), turned to 90 degrees
- moved JP1 5.89 mm to (88.5, 72.5)
- moved TP3 5.69 mm to (82.5, 75.5)
- moved TP2 5.59 mm to (65.0, 80.5)
- moved RV1 5.00 mm to (57.4, 65.0), turned to 90 degrees
- moved R3 2.60 mm to (66.9, 77.0)
- moved J2 2.27 mm to (94.5, 72.5)
Connections:
- U1 pad 4: Vin -> GND
- U1 pad 8: GND -> Vin
- U2 pad 4: Vin -> GND
- U2 pad 8: GND -> Vin
Routing:
- net Vin: track 125.8 -> 138.4 mm
- net DCycle: track 12.6 -> 19.9 mm
- net ExtDCycle: track 6.37 -> 11.9 mm
- net Net-(U1B--): track 25.4 -> 20.7 mm
- net Net-(JP1-C): track 11.7 -> 15.6 mm
- net Net-(U1A-+): track 18.4 -> 15.1 mm
- net Vout: track 16.8 -> 18.9 mm
- net GND: track 0.00 -> 0.78 mm

Commit message: A mi también matenme porfa
Routing:
- net Net-(U1B--): track 20.7 -> 25.9 mm
Changed lines of the file:
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@@
+	)
+	(segment
+		(start 82.5 77)
+		(end 81.594867 77.905133)
+		(width 0.5)
+		(layer "B.Cu")
+		(net 1)
+	)
+	(segment
+		(start 81.594867 77.905133)
+		(end 81.594867 80.42)
+		(width 0.5)
+		(layer "B.Cu")
+		(net 1)
 	)
 	(segment
@@
 		(start 76.643867 71.151)
 		(end 76.643867 76.563867)
+		(width 0.5)
+		(layer "B.Cu")
+		(net 1)
+	)
+	(segment
+		(start 82.5 75.5)
+		(end 82.5 77)
 		(width 0.5)
 		(layer "B.Cu")
@@
 		(min_thickness 0.25)
 		(filled_areas_thickness no)
-		(fill
+		(fill yes
 			(thermal_gap 0.5)
 			(thermal_bridge_width 0.5)
